File: proxima/proxima.kicad_sch (KiCad schematic)
At the start: 0 parts

Commit message: base schematic
Parts:
- added C1, C15, C17, C2, C20, C21, C24, C25, C26, C27, C3, C4, C46, C5: 100nF, A_HDJ_Library:C_0402_1005Metric, symbol Device:C
- added C10: 2.2uF, A_HDJ_Library:C_0402_1005Metric, symbol Device:C
- added C11, C12: 20pF, A_HDJ_Library:C_0402_1005Metric, symbol Device:C
- added C13, C14: 6.8pF, A_HDJ_Library:C_0402_1005Metric, symbol Device:C
- added C16: 10uF, Capacitor_SMD:C_0805_2012Metric, symbol Device:C
- added C18, C19, C44, C45: 22uF, Capacitor_SMD:C_0805_2012Metric, symbol Device:C
- added C43: 2.2uF, Capacitor_SMD:C_0805_2012Metric, symbol Device:C
- added C6, C7, C8: 1uF, A_HDJ_Library:C_0402_1005Metric, symbol Device:C
- added C9: 10uF, A_HDJ_Library:C_0402_1005Metric, symbol Device:C
- added Card1: TF-01A, easyeda2kicad:TF-SMD_TF-01A, symbol easyeda2kicad:TF-01A
- added FB1: FCM1608KF-601T03, Inductor_SMD:L_0603_1608Metric, symbol Device:FerriteBead
- added J1, J2, J3, J4, J5, J6, J7, J8: Conn_01x03, Connector_PinHeader_2.54mm:PinHeader_1x03_P2.54mm_Vertical, symbol Connector_Generic:Conn_01x03
- added J10, J11, J12, J9: Conn_01x02, Connector_PinHeader_2.54mm:PinHeader_1x02_P2.54mm_Vertical, symbol Connector_Generic:Conn_01x02
- added L1: 4.7uH, Inductor_SMD:L_Coilcraft_XxL4020, symbol Device:L
- added L3: 5.6uH, Inductor_SMD:L_Coilcraft_XxL4020, symbol Device:L
- added Q1, Q2, Q3, Q4: IRLML0030, Package_TO_SOT_SMD:SOT-23, symbol Transistor_FET:IRLML0030
- added R1, R2: 5.1K, A_HDJ_Library:R_0402_1005Metric, symbol Device:R
- added R10, R11, R12, R13, R14, R3, R8, R9: 10K, A_HDJ_Library:R_0402_1005Metric, symbol Device:R
- added R16: 100K, A_HDJ_Library:R_0402_1005Metric, symbol Device:R
- added R17: 22.1K, A_HDJ_Library:R_0402_1005Metric, symbol Device:R
- added R18, R19, R20, R21: 470 Ohm, A_HDJ_Library:R_0402_1005Metric, symbol Device:R
- added SW1, SW2: TS-1088-AR02016, easyeda2kicad:SW-SMD_L3.9-W3.0-P4.45, symbol ASM1166:TS-1088-AR02016
- added U1: STM32F722RETx, Package_QFP:LQFP-64_10x10mm_P0.5mm, symbol MCU_ST_STM32F7:STM32F722RETx
- added U2: BMP580, easyeda2kicad:LGA-10_L2.0-W2.0-P0.50-TL_BMP580, symbol easyeda2kicad:BMP580
- added U3: LSM6DSV16XTR, LSM6DSV16XTR:XDCR_LSM6DSV16XTR, symbol LSM6DSV16XTR:LSM6DSV16XTR
- added U4: AP63205WU, Package_TO_SOT_SMD:TSOT-23-6, symbol Regulator_Switching:AP63205WU
- added U5: LMR51430XFDDCR, LMR51430:SOT-23-THIN-6_DDC_TEX, symbol 2025-11-28_01-28-39:LMR51430XFDDCR
- added U6: BMM150, Package_CSP:WLCSP-12_1.56x1.56mm_P0.4mm, symbol Sensor_Magnetic:BMM150
- added U8: SX1262IMLTRT, Package_DFN_QFN:QFN-24-1EP_4x4mm_P0.5mm_EP2.6x2.6mm, symbol RF:SX1262IMLTRT
- added USB1: TYPE-C 16PIN 2MD(073), easyeda2kicad:USB-C-SMD_TYPE-C-6PIN-2MD-073, symbol ASM1166:TYPE-C16PIN2MD(073)
- added X1: Q13FC1350000400, easyeda2kicad:FC-135R_L3.2-W1.5, symbol ASM1166:Q13FC1350000400
- added X2: X322525MOB4SI, easyeda2kicad:CRYSTAL-SMD_4P-L3.2-W2.5-BL, symbol easyeda2kicad:X322525MOB4SI
Connections:
- new net: J11.2 (Pin_2), Q3.3 (D)
- new net: C17.2, L1.1, U4.5 (SW)
- new net: C17.1, U4.6 (BST)
- new net: R16.2, R17.2, U5.4 (FB)
- new net: FB1.2, U1.13 (VDDA)
- new net: R1.2, USB1.4 (CC1)
- new net: C46.2, L3.1, U5.2 (SW)
- new net: U8.2 (GND), U8.20 (GND), U8.25 (GND), U8.5 (GND), U8.8 (GND)
- new net: C46.1, U5.6 (CB)
- new net: R2.2, USB1.10 (CC2)
- new net: J12.2 (Pin_2), Q4.3 (D)
- new net: J9.2 (Pin_2), Q1.3 (D)
- new net: C10.1, U1.30 (VCAP_1)
- new net: J10.2 (Pin_2), Q2.3 (D)
- new net +3V3: C1.1, C2.1, C20.1, C21.1, C24.1, C25.1, C26.1, C27.1, C3.1, C4.1, C44.1, C45.1, C5.1, C6.1, C7.1, C8.1, C9.1, Card1.4 (VDD), FB1.1, L3.2, R10.2, R11.2, R12.2, R13.2, R14.1, R16.1, R8.2, R9.2, SW2.1, U1.1 (VBAT), U1.19 (VDD), U1.32 (VDD), U1.48 (VDD), U1.64 (VDD), U2.1 (VDDIO), U2.10 (VDD), U3.5 (VDD_IO), U3.8 (VDD), U6.A1 (PS), U6.B2 (VDDIO), U6.E5 (VDD)
- new net +5V: C18.1, C19.1, J1.2 (Pin_2), J2.2 (Pin_2), J3.2 (Pin_2), J4.2 (Pin_2), J5.2 (Pin_2), J6.2 (Pin_2), J7.2 (Pin_2), J8.2 (Pin_2), L1.2, U4.1 (FB)
- new net BARO_INT: U1.56 (PB4), U2.7 (INT)
- new net BOOT: R3.2, SW2.2, U1.60 (BOOT0)
- new net FIN_1: J5.1 (Pin_1), U1.37 (PC6)
- new net FIN_2: J6.1 (Pin_1), U1.38 (PC7)
- new net FIN_3: J7.1 (Pin_1), U1.25 (PB0)
- new net FIN_4: J8.1 (Pin_1), U1.26 (PB1)
- new net GND: C1.2, C10.2, C11.2, C12.2, C13.2, C14.2, C15.1, C16.2, C18.2, C19.2, C2.2, C20.2, C21.2, C24.2, C25.2, C26.2, C27.2, C3.2, C4.2, C43.1, C44.2, C45.2, C5.2, C6.2, C7.2, C8.2, C9.2, Card1.10 (GND), Card1.11 (GND), Card1.12 (GND), Card1.13 (GND), Card1.6 (VSS), J1.3 (Pin_3), J2.3 (Pin_3), J3.3 (Pin_3), J4.3 (Pin_3), J5.3 (Pin_3), J6.3 (Pin_3), J7.3 (Pin_3), J8.3 (Pin_3), Q1.2 (S), Q2.2 (S), Q3.2 (S), Q4.2 (S), R1.1, R17.1, R18.1, R19.1, R2.1, R20.1, R21.1, R3.1, SW1.1, U1.12 (VSSA), U1.18 (VSS), U1.31 (VSS), U1.47 (VSS), U1.63 (VSS), U2.3 (VSS), U2.5 (SDO), U2.6 (CSB), U2.8 (VSS), U2.9 (VSS), U3.6 (GND), U3.7 (GND__1), U4.4 (GND), U5.1 (GND), U6.A5 (CSB), U6.C1 (SDO), U6.C5 (GND), U6.E1 (GND), U6.E3 (GND), USB1.1 (GND), USB1.12 (GND), USB1.13 (SHELL), USB1.14 (SHELL), X2.2 (GND), X2.4 (GND)
- new net HSE_IN: C11.1, U1.5 (PH0), X2.1 (OSC1)
- new net HSE_OUT: C12.1, U1.6 (PH1), X2.3 (OSC2)
- new net I2C_SCL: U1.58 (PB6), U2.2 (SCK), U6.A3 (SCK)
- new net I2C_SDA: U1.59 (PB7), U2.4 (SDI), U6.B4 (SDI)
- new net IMU_CS: R14.2, U1.20 (PA4), U3.12 (CS)
- new net IMU_INT1: U1.41 (PA8), U3.4 (INT1)
- new net IMU_INT2: U1.42 (PA9), U3.9 (INT2)
- new net IMU_SCK: U1.21 (PA5), U3.13 (SCL)
- new net IMU_SDA: U1.23 (PA7), U3.14 (SDA)
- new net IMU_SDO: U1.22 (PA6), U3.1 (SDO/SA0)
- new net LSE_IN: C13.1, U1.3 (PC14), X1.1
- new net LSE_OUT: C14.1, U1.4 (PC15), X1.2
- new net MAG_INT: U1.57 (PB5), U6.D2 (INT)
- new net PYRO_1: Q1.1 (G), R19.2
- new net PYRO_2: Q2.1 (G), R18.2
- new net PYRO_3: Q3.1 (G), R20.2
- new net PYRO_4: Q4.1 (G), R21.2
- new net RESET: C15.2, SW1.2, U1.7 (NRST)
- new net SD_CD: Card1.9 (CD), U1.55 (PB3)
- new net SD_CMD: Card1.3 (CMD(DI)), R9.1, U1.54 (PD2)
- new net SD_DAT0: Card1.7 (DAT0(D0)), R13.1, U1.39 (PC8)
- new net SD_DAT1: Card1.8 (DAT1(RSV)), R12.1, U1.40 (PC9)
- new net SD_DAT2: Card1.1 (DAT2(RSV)), R11.1, U1.51 (PC10)
- new net SD_DAT3: Card1.2 (CDDAT3(CS)), R10.1, U1.52 (PC11)
- new net SD_SCLK: Card1.5 (CLK(SCLK)), R8.1, U1.53 (PC12)
- new net TVC_1: J1.1 (Pin_1), U1.14 (PA0)
- new net TVC_2: J2.1 (Pin_1), U1.15 (PA1)
- new net TVC_3: J4.1 (Pin_1), U1.16 (PA2)
- new net TVC_4: J3.1 (Pin_1), U1.17 (PA3)
- new net USB_DN: U1.44 (PA11), USB1.5 (DN2), USB1.7 (DN1)
- new net USB_DP: U1.45 (PA12), USB1.6 (DP1), USB1.8 (DP2)
- new net VBUS: USB1.11 (VBUS), USB1.2 (VBUS)
- new net VSYS: C16.1, C43.2, J10.1 (Pin_1), J11.1 (Pin_1), J12.1 (Pin_1), J9.1 (Pin_1), U4.2 (EN), U4.3 (IN), U5.3 (VIN), U5.5 (EN)
- no-connect marks 0 -> 2
